Commit message: feat: 完整的挖掘机智能避障系统源代码
- 感知模块：YOLOv5(COCO)+DeepSort跟踪+激光雷达处理+传感器融合+轨迹预测
- 风险评估：多因子加权评分(距离+TTC+类型权重)，LOW/MEDIUM/HIGH三级分类
- 决策模块：FSM状态机(NORMAL/CAUTION/PAUSED/EMERGENCY_STOP)
- 规划模块：改进RRT*路径规划(C++17，5次多项式平滑)
- 仿真验证：Gazebo 11，三个演示场景(G1/G2/G3)，all pass
- 监控面板：Flask+SSE Web Dashboard

验证通过：Phase 7 真实端到端Gazebo仿真，git tag v1.1-real-sim
可直接catkin_make编译使用，无需额外配置。

File: src/excavator_description/urdf/excavator.urdf.xacro (robot description, xacro)
@@ -66,10 +66,8 @@
       <xacro:box_inertia m="${track_mass}" x="${track_len}" y="${track_wid}" z="${track_hgt}"/>
     </link>
-    <joint name="${prefix}_track_joint" type="continuous">
+    <joint name="${prefix}_track_joint" type="fixed">
       <parent link="base_link"/>
       <child  link="${prefix}_track_link"/>
       <origin xyz="0 ${reflect * track_offset_y} ${-chassis_hgt/2 + track_hgt/2}" rpy="0 0 0"/>
-      <axis xyz="0 1 0"/>
-      <dynamics damping="0.1" friction="1.0"/>
     </joint>
     <gazebo reference="${prefix}_track_link">
@@ -253,23 +251,13 @@
   <!-- 传感器连杆、关节和 Gazebo 插件定义在 sensors.xacro 中 -->
   <xacro:include filename="$(find excavator_description)/urdf/sensors.xacro"/>
-  <!-- ===== Gazebo 插件：差速驱动 ===== -->
+  <!-- ===== Gazebo 插件：平面移动（planar_move） ===== -->
+  <!-- 方案B：替换 diff_drive，彻底绕开履带滚动物理问题（ADR-013） -->
   <gazebo>
-    <plugin name="differential_drive_controller" filename="libgazebo_ros_diff_drive.so">
-      <leftJoint>left_track_joint</leftJoint>
-      <rightJoint>right_track_joint</rightJoint>
-      <wheelSeparation>${2 * track_offset_y}</wheelSeparation>
-      <wheelDiameter>${track_hgt}</wheelDiameter>
-      <wheelTorque>20000</wheelTorque>
-      <wheelAcceleration>1.0</wheelAcceleration>
+    <plugin name="planar_move_controller" filename="libgazebo_ros_planar_move.so">
       <commandTopic>cmd_vel</commandTopic>
       <odometryTopic>odom</odometryTopic>
       <odometryFrame>odom</odometryFrame>
+      <odometryRate>20.0</odometryRate>
       <robotBaseFrame>base_footprint</robotBaseFrame>
-      <odometrySource>1</odometrySource>
-      <publishWheelTF>false</publishWheelTF>
-      <publishOdomTF>true</publishOdomTF>
-      <!-- 关闭 wheel joint state 发布；由 joint_state_publisher 统一发布全部关节，避免双写 /joint_states -->
-      <publishWheelJointState>false</publishWheelJointState>
-      <legacyMode>false</legacyMode>
     </plugin>
   </gazebo>
