Commit message: fix(planner): G3 综合修复 — ADR-029/030/031 (robot_radius + cluster offset + path cleanup)
本 commit 累计 ADR-023 ~ ADR-031 全部改动（自上次 commit 67fa85a 之后的全部修复）。

主线问题修复（2026-05-21）：
- ADR-029: rrt_star_planner 引入 robot_radius 圆盘机器人模型替代 point inflation
  解决"矩形车体角部 3.61m vs 排除圆 2.5m"几何不匹配 → 转弯卡死
- ADR-030: goalCb 不提前清旧 path，plan 失败时保留 fallback
  解决"2D Nav Goal 接收新目标但 plan 失败时机器人停滞"
- ADR-031: obstacleCb 加 LIDAR_FACE_BIAS=0.5m 反向偏移修正 cluster 中心；
  goal reached / plan failed 时发布空 nav_msgs::Path 让 RViz 清除显示
  解决"偶发碰撞 + RViz 路径走完不消失 + 用户点 goal 无视觉反馈"

辅助 ADR（2026-05-20）：
- ADR-023: urdf 手臂收起（boom/arm/bucket rpy）
- ADR-025: fsm_controller CAUTION 速度恢复正常
- ADR-028: test_static.world 回退至 ADR-019 三障碍布局

最终生效参数: robot_radius=3.5, obstacle_margin=0.3, goal_x=24.0

验证 (WSL Gazebo+RViz, sim_time 50s+):
- G3 端到端: spawn(0,0) -> goal(24,0), goal reached @36s, dist=0.231m
- 0 次 EMERGENCY_STOP, 0 次碰撞卡死
- 不可达 goal 测试: 机器人按 fallback 继续走
- goal reached 后 /planned_path poses=0 (RViz 自动清除)

详见 tasks/decisions.md ADR-023 ~ ADR-031 完整记录。

File: src/excavator_description/urdf/excavator_simple.urdf.xacro (robot description, xacro)
@@ -35,8 +35,8 @@
       <material name="dark_gray"/>
     </visual>
-    <collision>
+      <collision>
       <geometry><box size="${chassis_len} ${chassis_wid} ${chassis_hgt}"/></geometry>
     </collision>
-    <xacro:box_inertia m="${chassis_mass}" x="${chassis_len}" y="${chassis_wid}" z="${chassis_hgt}"/>
+        <xacro:box_inertia m="${chassis_mass}" x="${chassis_len}" y="${chassis_wid}" z="${chassis_hgt}"/>
   </link>
   <gazebo reference="base_link">
@@ -55,5 +55,5 @@
       <geometry><box size="3.0 2.2 0.9"/></geometry>
     </collision>
-    <xacro:box_inertia m="1800.0" x="3.0" y="2.2" z="0.9"/>
+        <xacro:box_inertia m="1800.0" x="3.0" y="2.2" z="0.9"/>
   </link>
   <joint name="turret_joint" type="fixed">
@@ -73,9 +73,9 @@
     <parent link="turret_link"/>
     <child link="boom_link"/>
-    <origin xyz="1.0 0 0.35" rpy="0 0 0"/>
+    <origin xyz="1.0 0 0.35" rpy="0 -1.05 0"/>
   </joint>
   <link name="arm_link">
     <visual>
-      <origin xyz="1.0 0 -0.15" rpy="0 0.35 0"/>
+      <origin xyz="1.0 0 -0.15" rpy="0 0 0"/>
       <geometry><box size="2.2 0.25 0.25"/></geometry>
       <material name="excavator_yellow"/>
@@ -86,5 +86,5 @@
     <parent link="boom_link"/>
     <child link="arm_link"/>
-    <origin xyz="3.2 0 0.0" rpy="0 0 0"/>
+    <origin xyz="3.2 0 0.0" rpy="0 2.62 0"/>
   </joint>
   <link name="bucket_link">
@@ -99,5 +99,5 @@
     <parent link="arm_link"/>
     <child link="bucket_link"/>
-    <origin xyz="2.0 0 -0.1" rpy="0 0 0"/>
+    <origin xyz="2.0 0 -0.1" rpy="0 -0.52 0"/>
   </joint>
   <link name="sensor_mast_link">
